Commit message: add imu sensor

File: assets/xacro/base.mujoco.xacro (robot description, xacro)
@@ -45,7 +45,4 @@
   <xacro:macro name="base" params="name">
     <worldbody>
-        <body name="test" pos="0 0 0.5">
-          <geom name="wheel_test" type="mesh" rgba="0.1 0.1 0.1 1" mesh="wheel" />
-        </body>
         <light name="spotlight" mode="targetbodycom" target="${name}_link" pos="0 -1 2" cutoff="30"/>
         <body name="${name}_link" pos="0 0 0.11" quat="1 0 0 0" >
@@ -53,4 +50,5 @@
             <inertial mass="28" pos="0 0 0.0515" fullinertia="0.465408937 0.483193291 0.550939703 0.002160024 -0.001760255 -0.000655952"/>
             <body name="base_footprint" pos="0 0 ${wheel_radius}" />
+            <site name="${name}_imu_site"/>
             <geom pos="0 0 0.0985" type="mesh" rgba="1 1 1 1"     mesh="base"/>
             <geom pos="-0.183 0.183 0.173"  quat=" 0.382683 0 0 0.92388" type="mesh" rgba="0.1 0.1 0.1 1" mesh="srf05"/>
@@ -83,14 +81,8 @@
         <exclude body1="wheel_left_link"  body2="${name}_link"/>
     </contact>
-    <tendon>
-      <fixed name="forward">
-        <joint joint="wheel_left_joint" coef="1.5"/>
-        <joint joint="wheel_right_joint" coef="1.5"/>
-      </fixed>
-      <fixed name="turn">
-        <joint joint="wheel_left_joint" coef="-1.5"/>
-        <joint joint="wheel_right_joint" coef="1.5"/>
-      </fixed>
-    </tendon>
+    <sensor>
+      <accelerometer name="${name}_linear_acc_sensor" site="${name}_imu_site"/>
+      <gyro name="${name}_angular_vel_sensor" site="${name}_imu_site"/>
+    </sensor>
   </xacro:macro>
 </mujoco>

Commit message: add floor and set friction

File: assets/xacro/base.mujoco.xacro (robot description, xacro)
@@ -46,5 +46,5 @@
     <worldbody>
         <light name="spotlight" mode="targetbodycom" target="${name}_link" pos="0 -1 2" cutoff="30"/>
-        <body name="${name}_link" pos="0 0 0.11" quat="1 0 0 0" >
+        <body name="${name}_link" pos="0 0 0.21" quat="1 0 0 0" >
             <freejoint/>
             <inertial mass="28" pos="0 0 0.0515" fullinertia="0.465408937 0.483193291 0.550939703 0.002160024 -0.001760255 -0.000655952"/>

File: example/scene.xml.xacro (robot description, xacro)
@@ -1,23 +1,26 @@
 <?xml version="1.0"?>
-<mujoco xmlns:xacro="http://ros.org/wiki/xacro"
-        model="pmb2 Scene" >
+<mujoco xmlns:xacro="http://ros.org/wiki/xacro" model="pmb2 Scene">
   <xacro:include filename="$(find pmb2_mujoco)/assets/xacro/pmb2.mujoco.xacro" />
   <statistic center="0 0 0.3" extent="1.2"/>
   <visual>
-    <headlight diffuse="0.6 0.6 0.6"  ambient="0.3 0.3 0.3" specular="0 0 0"/>
+    <headlight diffuse="0.6 0.6 0.6" ambient="0.3 0.3 0.3" specular="0 0 0"/>
     <rgba haze="0.15 0.25 0.35 1"/>
     <global azimuth="120" elevation="-20"/>
   </visual>
   <asset>
-    <texture type="skybox" builtin="gradient" rgb1="0.3 0.5 0.7" rgb2="0 0 0" width="512"
-        height="3072"/>
-    <texture type="2d" name="groundplane" builtin="checker" mark="edge" rgb1="0.2 0.3 0.4"
-        rgb2="0.1 0.2 0.3" markrgb="0.8 0.8 0.8" width="300" height="300"/>
-    <material name="groundplane" texture="groundplane" texuniform="true" texrepeat="5 5"
-        reflectance="0.2"/>
+    <texture type="skybox" builtin="gradient" rgb1="0.3 0.5 0.7" rgb2="0 0 0" width="512" height="3072"/>
+    <texture type="2d" name="groundplane" builtin="checker" mark="edge" rgb1="0.2 0.3 0.4" rgb2="0.1 0.2 0.3" markrgb="0.8 0.8 0.8" width="300" height="300"/>
+    <material name="groundplane" texture="groundplane" texuniform="true" texrepeat="5 5" reflectance="0.2"/>
+    <texture name="grid" type="2d" builtin="checker" width="512" height="512" rgb1=".1 .2 .3" rgb2=".2 .3 .4"/>
+    <material name="grid" texture="grid" texrepeat="1 1" texuniform="true" reflectance=".2"/>
   </asset>
   <worldbody>
     <light pos="0 0 1.5" dir="0 0 -1" directional="true"/>
     <geom name="floor" size="0 0 0.05" type="plane" material="groundplane"/>
+    <geom name="low_friction0" type="box" pos="0 0 0.1" size="400 400 .01" material="grid" condim="3"/>
   </worldbody>
+  <contact>
+    <pair geom1="wheel_left" geom2="low_friction0" friction="0.1 0.1 0.005 0.0001 0.0001"/>
+    <pair geom1="wheel_right" geom2="low_friction0" friction="0.1 0.1 0.005 0.0001 0.0001"/>
+  </contact>
 </mujoco>

Commit message: Split definitions into individual macros

File: assets/xacro/base.mujoco.xacro (robot description, xacro)
@@ -1,28 +1,6 @@
 <?xml version="1.0"?>
-<!--
-  Copyright (c) 2021 PAL Robotics S.L. All rights reserved.
-  Licensed under the Apache License, Version 2.0 (the "License");
-  you may not use this file except in compliance with the License.
-  You may obtain a copy of the License at
-      http://www.apache.org/licenses/LICENSE-2.0
-  Unless required by applicable law or agreed to in writing, software
-  distributed under the License is distributed on an "AS IS" BASIS,
-  WITHOUT WARRANTIES OR CONDITIONS OF ANY KIND, either express or implied.
-  See the License for the specific language governing permissions and
-  limitations under the License.
--->
 <mujoco xmlns:xacro="http://ros.org/wiki/xacro">
   <compiler angle="radian" meshdir="$(find pmb2_description)/meshes/" autolimits="false"/>
   <size njmax="500" nconmax="100"/>
-  <asset>
-    <mesh name="sick_tim551" file="sensors/sick_tim551.stl"/>
-    <mesh name="srf05" file="sensors/srf05.stl"/>
-    <mesh name="base" file="base/base.stl" refpos="0 0 0.0985" />
-    <mesh name="base_ring" file="base/base_ring.stl"/>
-    <mesh name="antenna" file="objects/antenna.stl"/>
-    <mesh name="wheel" file="wheels/wheel.stl"/>
-    <mesh name="caster_1" file="wheels/caster_1.stl"/>
-    <mesh name="caster_2" file="wheels/caster_2.stl"/>
-  </asset>
   <xacro:include filename="$(find pmb2_mujoco)/assets/xacro/wheel.mujoco.xacro"/>
   <xacro:include filename="$(find pmb2_mujoco)/assets/xacro/caster.mujoco.xacro"/>
@@ -43,46 +21,29 @@
   <xacro:property name="caster_offset_y"     value="0.0"/>
   <xacro:property name="caster_offset_z"     value="-0.0335"/>
-  <xacro:macro name="base" params="name">
-    <worldbody>
-        <light name="spotlight" mode="targetbodycom" target="${name}_link" pos="0 -1 2" cutoff="30"/>
-        <body name="${name}_link" pos="0 0 0.21" quat="1 0 0 0" >
-            <freejoint/>
-            <inertial mass="28" pos="0 0 0.0515" fullinertia="0.465408937 0.483193291 0.550939703 0.002160024 -0.001760255 -0.000655952"/>
-            <body name="base_footprint" pos="0 0 ${wheel_radius}" />
-            <site name="${name}_imu_site"/>
-            <geom pos="0 0 0.0985" type="mesh" rgba="1 1 1 1"     mesh="base"/>
-            <geom pos="-0.183 0.183 0.173"  quat=" 0.382683 0 0 0.92388" type="mesh" rgba="0.1 0.1 0.1 1" mesh="srf05"/>
-            <geom pos="-0.183 -0.183 0.173" quat="-0.382683 0 0 0.92388" type="mesh" rgba="0.1 0.1 0.1 1" mesh="srf05"/>
-            <geom pos="-0.259 0 0.173"      quat="0 0 0 1"               type="mesh" rgba="0.1 0.1 0.1 1" mesh="srf05"/>
-            <geom pos=" 0.202 0 -0.004"                                  type="mesh" rgba="0.1 0.1 0.1 1" mesh="sick_tim551"/>
-            <geom pos="0 0 0.0315" type="mesh" rgba="1 0.487 0 1" mesh="base_ring"/>
-            <xacro:antenna name="${name}_antenna_left"  xyz="-0.201  0.1062 0.195" rpy="0 0 0" />
-            <xacro:antenna name="${name}_antenna_right" xyz="-0.201 -0.1062 0.195" rpy="0 0 0" />
-            <!-- Wheels -->
-            <xacro:wheel side="right" reflect=" 1.0" radius="${wheel_radius}" width="${wheel_width}" torque="${wheel_torque}" velocity="${wheel_velocity}" separation="${wheel_separation}" />
-            <xacro:wheel side="left"  reflect="-1.0" radius="${wheel_radius}" width="${wheel_width}" torque="${wheel_torque}" velocity="${wheel_velocity}" separation="${wheel_separation}" />
-            <!-- Casters wheels -->
-            <xacro:caster side="front_right" radius="${caster_radius}" width="${caster_width}" separation_x="${ caster_separation_x}" separation_y="${ caster_separation_y}" offset_x="${caster_offset_x}" offset_y="${caster_offset_y}" offset_z="${caster_offset_z}" />
-            <xacro:caster side="front_left"  radius="${caster_radius}" width="${caster_width}" separation_x="${ caster_separation_x}" separation_y="${-caster_separation_y}" offset_x="${caster_offset_x}" offset_y="${caster_offset_y}" offset_z="${caster_offset_z}" />
-            <xacro:caster side="back_right"  radius="${caster_radius}" width="${caster_width}" separation_x="${-caster_separation_x}" separation_y="${ caster_separation_y}" offset_x="${caster_offset_x}" offset_y="${caster_offset_y}" offset_z="${caster_offset_z}" />
-            <xacro:caster side="back_left"   radius="${caster_radius}" width="${caster_width}" separation_x="${-caster_separation_x}" separation_y="${-caster_separation_y}" offset_x="${caster_offset_x}" offset_y="${caster_offset_y}" offset_z="${caster_offset_z}" />
-        </body>
-    </worldbody>
-    <contact>
-        <exclude body1="caster_front_right_1_link" body2="${name}_link"/>
-        <exclude body1="caster_front_left_1_link"  body2="${name}_link"/>
-        <exclude body1="caster_back_right_1_link"  body2="${name}_link"/>
-        <exclude body1="caster_back_left_1_link"   body2="${name}_link"/>
-        <exclude body1="caster_front_right_2_link" body2="${name}_link"/>
-        <exclude body1="caster_front_left_2_link"  body2="${name}_link"/>
-        <exclude body1="caster_back_right_2_link"  body2="${name}_link"/>
-        <exclude body1="caster_back_left_2_link"   body2="${name}_link"/>
-        <exclude body1="wheel_right_link" body2="${name}_link"/>
-        <exclude body1="wheel_left_link"  body2="${name}_link"/>
-    </contact>
-    <sensor>
-      <accelerometer name="${name}_linear_acc_sensor" site="${name}_imu_site"/>
-      <gyro name="${name}_angular_vel_sensor" site="${name}_imu_site"/>
-    </sensor>
+  <xacro:macro name="base" params="name pos quat *attached_body">
+      <light name="spotlight" mode="targetbodycom" target="${name}_link" pos="0 -1 2" cutoff="30"/>
+      <body name="${name}_link" pos="${pos}" quat="${quat}" >
+          <freejoint/>
+          <inertial mass="28" pos="0 0 0.0515" fullinertia="0.465408937 0.483193291 0.550939703 0.002160024 -0.001760255 -0.000655952"/>
+          <xacro:insert_block name="attached_body" />
+          <body name="base_footprint" pos="0 0 ${wheel_radius}" />
+          <site name="${name}_imu_site"/>
+          <geom pos="0 0 0.0985" type="mesh" rgba="1 1 1 1"     mesh="base"/>
+          <geom pos="-0.183 0.183 0.173"  quat=" 0.382683 0 0 0.92388" type="mesh" rgba="0.1 0.1 0.1 1" mesh="srf05"/>
+          <geom pos="-0.183 -0.183 0.173" quat="-0.382683 0 0 0.92388" type="mesh" rgba="0.1 0.1 0.1 1" mesh="srf05"/>
+          <geom pos="-0.259 0 0.173"      quat="0 0 0 1"               type="mesh" rgba="0.1 0.1 0.1 1" mesh="srf05"/>
+          <geom pos=" 0.202 0 -0.004"                                  type="mesh" rgba="0.1 0.1 0.1 1" mesh="sick_tim551"/>
+          <geom pos="0 0 0.0315" type="mesh" rgba="1 0.487 0 1" mesh="base_ring"/>
+          <xacro:antenna name="${name}_antenna_left"  xyz="-0.201  0.1062 0.195" rpy="0 0 0" />
+          <xacro:antenna name="${name}_antenna_right" xyz="-0.201 -0.1062 0.195" rpy="0 0 0" />
+          <!-- Wheels -->
+          <xacro:wheel side="right" reflect=" 1.0" radius="${wheel_radius}" width="${wheel_width}" torque="${wheel_torque}" velocity="${wheel_velocity}" separation="${wheel_separation}" />
+          <xacro:wheel side="left"  reflect="-1.0" radius="${wheel_radius}" width="${wheel_width}" torque="${wheel_torque}" velocity="${wheel_velocity}" separation="${wheel_separation}" />
+          <!-- Casters wheels -->
+          <xacro:caster side="front_right" radius="${caster_radius}" width="${caster_width}" separation_x="${ caster_separation_x}" separation_y="${ caster_separation_y}" offset_x="${caster_offset_x}" offset_y="${caster_offset_y}" offset_z="${caster_offset_z}" />
+          <xacro:caster side="front_left"  radius="${caster_radius}" width="${caster_width}" separation_x="${ caster_separation_x}" separation_y="${-caster_separation_y}" offset_x="${caster_offset_x}" offset_y="${caster_offset_y}" offset_z="${caster_offset_z}" />
+          <xacro:caster side="back_right"  radius="${caster_radius}" width="${caster_width}" separation_x="${-caster_separation_x}" separation_y="${ caster_separation_y}" offset_x="${caster_offset_x}" offset_y="${caster_offset_y}" offset_z="${caster_offset_z}" />
+          <xacro:caster side="back_left"   radius="${caster_radius}" width="${caster_width}" separation_x="${-caster_separation_x}" separation_y="${-caster_separation_y}" offset_x="${caster_offset_x}" offset_y="${caster_offset_y}" offset_z="${caster_offset_z}" />
+      </body>
   </xacro:macro>
 </mujoco>

File: assets/xacro/pmb2.mujoco.xacro (robot description, xacro)
@@ -12,9 +12,7 @@
   limitations under the License.
 -->
-<mujoco  xmlns:xacro="http://ros.org/wiki/xacro"
-        model="pmb2" >
+<mujoco xmlns:xacro="http://ros.org/wiki/xacro" model="pmb2" >
   <xacro:arg name="laser_model" default="sick-571"/> <!-- false, hokuyo, sick-551, sick-561, sick-571-->
   <xacro:arg name="rgbd_sensors" default="false"/> <!-- false, true-->
-  <xacro:arg name="name" default="pmb2" />
   <xacro:property name="laser_model" value="$(arg laser_model)" />
   <xacro:property name="rgbd_sensors" value="$(arg rgbd_sensors)"/>
@@ -27,5 +25,9 @@
   <xacro:property name="nsp" value="$(arg namespace)" />
   <xacro:include filename="$(find pmb2_mujoco)/assets/xacro/base.mujoco.xacro" />
-  <xacro:base name="$(arg name)" />
+  <xacro:macro name="pmb2_robot" params="name pos quat *attached_body">
+    <xacro:base name="${name}" pos="${pos}" quat="${quat}" >
+      <xacro:insert_block name="attached_body" />
+    </xacro:base>
+  </xacro:macro>
   <!-- The following included files set up definitions of parts of the robot body -->
   <!-- Base -->

File: example/scene.xml.xacro (robot description, xacro)
@@ -2,4 +2,8 @@
 <mujoco xmlns:xacro="http://ros.org/wiki/xacro" model="pmb2 Scene">
   <xacro:include filename="$(find pmb2_mujoco)/assets/xacro/pmb2.mujoco.xacro" />
+  <xacro:include filename="$(find pmb2_mujoco)/assets/xacro/assets.mujoco.xacro" />
+  <xacro:include filename="$(find pmb2_mujoco)/assets/xacro/contacts.mujoco.xacro" />
+  <xacro:include filename="$(find pmb2_mujoco)/assets/xacro/sensors.mujoco.xacro" />
+  <xacro:pmb2_assets />
   <statistic center="0 0 0.3" extent="1.2"/>
   <visual>
@@ -20,4 +24,11 @@
     <geom name="low_friction0" type="box" pos="0 0 0.1" size="400 400 .01" material="grid" condim="3"/>
   </worldbody>
+  <worldbody>
+    <xacro:pmb2_robot name="pmb2" pos="0 0 0.21" quat="1 0 0 0" >
+      <body />
+    </xacro:pmb2_robot>
+  </worldbody>
+  <xacro:pmb2_contacts name="pmb2" />
+  <xacro:pmb2_sensors name="pmb2" />
   <contact>
     <pair geom1="wheel_left" geom2="low_friction0" friction="0.1 0.1 0.005 0.0001 0.0001"/>

Commit message: fixes quat/rot naming convention in xacro files

File: assets/xacro/base.mujoco.xacro (robot description, xacro)
@@ -19,7 +19,7 @@
   <xacro:property name="caster_offset_y"     value="0.0"/>
   <xacro:property name="caster_offset_z"     value="-0.0335"/>
-  <xacro:macro name="base" params="name pos quat *attached_body">
+  <xacro:macro name="base" params="name pos rot *attached_body">
       <light name="spotlight" mode="targetbodycom" target="${name}_link" pos="0 -1 2" cutoff="30"/>
-      <body name="${name}_link" pos="${pos}" quat="${quat}" >
+      <body name="${name}_link" pos="${pos}" euler="${rot}" >
           <freejoint/>
           <inertial mass="28" pos="0 0 0.0515" fullinertia="0.465408937 0.483193291 0.550939703 0.002160024 -0.001760255 -0.000655952"/>

File: assets/xacro/pmb2.mujoco.xacro (robot description, xacro)
@@ -25,6 +25,6 @@
   <xacro:property name="nsp" value="$(arg namespace)" />
   <xacro:include filename="$(find pmb2_mujoco)/assets/xacro/base.mujoco.xacro" />
-  <xacro:macro name="pmb2_robot" params="name pos quat *attached_body">
-    <xacro:base name="${name}" pos="${pos}" quat="${quat}" >
+  <xacro:macro name="pmb2_robot" params="name pos rot *attached_body">
+    <xacro:base name="${name}" pos="${pos}" rot="${rot}" >
       <xacro:insert_block name="attached_body" />
     </xacro:base>
