Commit message: wip: tiago tuning

File: pmb2_mujoco/assets/xacro/base.mujoco.xacro (robot description, xacro)
@@ -23,5 +23,5 @@
       <body name="${name}_link" pos="${pos}" euler="${rot}" >
           <freejoint/>
-          <inertial mass="28" pos="0 0 0.0515" fullinertia="0.465408937 0.483193291 0.550939703 0.002160024 -0.001760255 -0.000655952"/>
+          <inertial mass="55" pos="0 0 -0.0515" diaginertia="1 1 1"/>
           <xacro:insert_block name="attached_body" />
           <body name="base_footprint" pos="0 0 ${wheel_radius}" />

File: pmb2_mujoco/assets/xacro/caster.mujoco.xacro (robot description, xacro)
@@ -4,10 +4,10 @@
     <body name="caster_${side}_1_link" pos="${offset_x + separation_x / 2} ${offset_y - separation_y / 2} ${offset_z}">
         <inertial pos="-0.00634599 5.347e-05 -0.0203752" mass="0.0514476" fullinertia="0.00001513 0.00001309 0.00001198 -0.00000003 0.00000267 -0.00000005"/>
-        <joint name="caster_${side}_1_joint" pos="0 0 0" axis="0 0 1" damping="0.005"/>
+        <joint name="caster_${side}_1_joint" pos="0 0 0" axis="0 0 1" damping="0.005" frictionloss="50.0"/>
         <geom type="mesh" rgba="0.7 0.7 0.7 1" mesh="caster_1"/>
         <body name="caster_${side}_2_link" pos="-0.016 0 -0.04" euler="${-90.0/180*pi} 0 0">
-            <inertial pos="0 0 0" euler="0 0 0" mass="0.0885578" diaginertia="1.075e-05 1.541e-05 1.075e-05"/>
+            <inertial pos="0 0 0" euler="0 0 0" mass="0.0885578" diaginertia="1.541e-05 1.541e-05 1.541e-05"/>
             <joint name="caster_${side}_2_joint" pos="0 0 0" axis="0 0 1"/>
-            <geom type="mesh" rgba="0.1 0.1 0.1 1" mesh="caster_2"/>
+            <geom type="mesh" rgba="0.1 0.1 0.1 1" mesh="caster_2" friction="1 0.005 0.0001"/>
         </body>
     </body>

File: pmb2_mujoco/assets/xacro/wheel.mujoco.xacro (robot description, xacro)
@@ -4,9 +4,9 @@
     <body name="suspension_${side}_link" pos="0 0 0">
         <inertial pos="0 0 -0.02" mass="0.1" diaginertia="1 1 1"/>
-        <joint name="suspension_${side}_joint" pos="0 0 0" axis="0 0 1" type="slide" frictionloss="0.001" stiffness="1000.0" springref="-0.12" damping="12.5"/>
+        <joint name="suspension_${side}_joint" pos="0 0 0" axis="0 0 1" type="slide" frictionloss="0.001" stiffness="5000.0" springref="-0.02" damping="12.5"/>
         <body name="wheel_${side}_link" pos="0 ${-0.2022 * reflect} 0" euler="${-90 /180*pi} 0 0">
             <inertial pos="0 0 ${-0.0207 * reflect}" mass="1.82362" fullinertia="0.00499743171 0.00499741733 0.00839239692 ${ 0.00000004464 * reflect} -0.00000002245 ${-0.00000000164 * reflect}"/>
             <joint name="wheel_${side}_joint" pos="0 0 0" axis="0 0 1"/>
-            <geom name="wheel_${side}" type="mesh" rgba="0.1 0.1 0.1 1" mesh="wheel" />
+            <geom name="wheel_${side}" type="mesh" rgba="0.1 0.1 0.1 1" mesh="wheel" friction="1 0.005 0.0001" />
         </body>
     </body>
